File: custom-boards/v1/kicad/Remapper.kicad_sch (KiCad schematic)
At the start: 57 parts, among them SW102 SW_Push, SW2 SW_Push, U103 RP2040, U105 W25Q128JVS, U3 RP2040, U4 TLV73333PDBV, U5 W25Q128JVS, Y1 Crystal_GND24, Y101 Crystal_GND24

Commit message: Update custom boards
This commit makes the following changes to the custom PCB designs.

v1-v5: flash chip footprint changed, previous one caused issues in
manufacturing. Some other components moved around as a result.

v1-v5: flash chip changed from 1 megabyte to 2 megabyte one.

v1: USB Type A port component changed, previous one was consistently
soldered on crooked by JLCPCB.

The new designs are named v1.1-v5.1.

Schematics and enclosure files are unchanged.
Parts:
- U105, U5: LCSC C401667 -> C2843335
- U4: footprint Package_TO_SOT_SMD:SOT-23-5 -> SOT:SOT-23-5
- USB1: footprint Type-A:908-261A2021S10100 -> Type-A:C42459; LCSC C39423 -> C42459
