File: custom-boards/v2/kicad/Remapper.kicad_sch (KiCad schematic)
At the start: 49 parts, among them J1 Conn_01x06, J101 Conn_01x06, U103 RP2040, U105 W25Q128JVS, U3 RP2040, U4 TLV73333PDBV, U5 W25Q128JVS, Y1 Crystal_GND24, Y101 Crystal_GND24

Commit message: Update custom boards
This commit makes the following changes to the custom PCB designs.

v1-v5: flash chip footprint changed, previous one caused issues in
manufacturing. Some other components moved around as a result.

v1-v5: flash chip changed from 1 megabyte to 2 megabyte one.

v1: USB Type A port component changed, previous one was consistently
soldered on crooked by JLCPCB.

The new designs are named v1.1-v5.1.

Schematics and enclosure files are unchanged.
Parts:
- J1, J101: now left out of the parts list
- U105, U5: LCSC C401667 -> C2843335
- U4: footprint Package_TO_SOT_SMD:SOT-23-5 -> SOT:SOT-23-5
