File: custom-boards/v4/kicad/Remapper.kicad_sch (KiCad schematic)
At the start: 46 parts, among them J1 AudioJack3, J2 AudioJack3, J3 AudioJack3, J4 AudioJack3, J5 AudioJack3, J6 AudioJack3, J7 AudioJack3, J8 AudioJack3, SW102 SW_Push, U103 RP2040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

Commit message: Update custom boards
This commit makes the following changes to the custom PCB designs.

v1-v5: flash chip footprint changed, previous one caused issues in
manufacturing. Some other components moved around as a result.

v1-v5: flash chip changed from 1 megabyte to 2 megabyte one.

v1: USB Type A port component changed, previous one was consistently
soldered on crooked by JLCPCB.

The new designs are named v1.1-v5.1.

Schematics and enclosure files are unchanged.
Parts:
- U105: LCSC C401667 -> C2843335
Changed lines of the file:
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@@
       (effects (font (size 1.27 1.27)) hide)
     )
-    (property "LCSC" "C401667" (at 240.03 144.78 0)
+    (property "LCSC" "C2843335" (at 240.03 144.78 0)
       (effects (font (size 1.27 1.27)) hide)
     )
