File: custom-boards/v5/kicad/Remapper.kicad_sch (KiCad schematic)
At the start: 67 parts, among them SW102 SW_Push, U1 SL2.1A, U103 RP2040, U105 W25Q128JVS, U3 RP2040, U4 TLV73333PDBV, U5 W25Q128JVS, Y1 Crystal_GND24, Y101 Crystal_GND24

Commit message: Update custom boards
This commit makes the following changes to the custom PCB designs.

v1-v5: flash chip footprint changed, previous one caused issues in
manufacturing. Some other components moved around as a result.

v1-v5: flash chip changed from 1 megabyte to 2 megabyte one.

v1: USB Type A port component changed, previous one was consistently
soldered on crooked by JLCPCB.

The new designs are named v1.1-v5.1.

Schematics and enclosure files are unchanged.
Parts:
- U105, U5: LCSC C401667 -> C2843335
Changed lines of the file:
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@@
       (effects (font (size 1.27 1.27)) hide)
     )
-    (property "LCSC" "C401667" (at 172.72 158.75 0)
+    (property "LCSC" "C2843335" (at 172.72 158.75 0)
       (effects (font (size 1.27 1.27)) hide)
     )
@@
       (effects (font (size 1.27 1.27)) hide)
     )
-    (property "LCSC" "C401667" (at 363.22 162.56 0)
+    (property "LCSC" "C2843335" (at 363.22 162.56 0)
       (effects (font (size 1.27 1.27)) hide)
     )
