File: custom-boards/v3/kicad/Remapper.kicad_sch (KiCad schematic)
At the start: 30 parts, among them SW102 SW_Push, U103 RP2040, U105 W25Q128JVS, U4 TLV73333PDBV, Y101 Crystal_GND24

Commit message: Update custom boards
This commit makes the following changes to the custom PCB designs.

v1-v5: flash chip footprint changed, previous one caused issues in
manufacturing. Some other components moved around as a result.

v1-v5: flash chip changed from 1 megabyte to 2 megabyte one.

v1: USB Type A port component changed, previous one was consistently
soldered on crooked by JLCPCB.

The new designs are named v1.1-v5.1.

Schematics and enclosure files are unchanged.
Parts:
- U105: LCSC C401667 -> C2843335
Changed lines of the file:
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@@
       (effects (font (size 1.27 1.27)) hide)
     )
-    (property "LCSC" "C401667" (at 204.47 147.32 0)
+    (property "LCSC" "C2843335" (at 204.47 147.32 0)
       (effects (font (size 1.27 1.27)) hide)
     )

Commit message: Add an LED to v3
Parts:
- added D1: LED, LED_SMD:LED_0201_0603Metric, symbol Device:LED
- added R108: 300, Resistor_SMD:R_0402_1005Metric, symbol Device:R
Connections:
- net GND: now also R108.2
- net L0: now reaches U103.29 (GPIO18)
- net L0: now also D1.2 (A)
- new net: D1.1 (K), R108.1
- no-connect marks 31 -> 30

Commit message: Use a cheaper type of LED
Parts:
- D1: footprint LED_SMD:LED_0201_0603Metric -> LED_SMD:LED_0402_1005Metric
Changed lines of the file:
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@@
 			)
 		)
-		(property "Footprint" "LED_SMD:LED_0201_0603Metric"
+		(property "Footprint" "LED_SMD:LED_0402_1005Metric"
 			(at 255.27 129.54 0)
 			(effects

Commit message: Use GPIO 19 instead of 18
Connections:
- net L0: now also U103.30 (GPIO19); no longer U103.29 (GPIO18)
Changed lines of the file:
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@@
-	)
-	(no_connect
-		(at 102.87 121.92)
 	)
 	(no_connect
@@
 	)
 	(no_connect
+		(at 102.87 119.38)
+	)
+	(no_connect
 		(at 102.87 83.82)
 	)
@@
 	(wire
 		(pts
-			(xy 107.95 127) (xy 107.95 119.38)
+			(xy 107.95 127) (xy 107.95 121.92)
 		)
 		(stroke
@@
 	(wire
 		(pts
-			(xy 107.95 119.38) (xy 102.87 119.38)
-		)
-		(stroke
+			(xy 107.95 121.92) (xy 102.87 121.92)
+		)
+		(stroke
